File: KiCAD/CIB - Star-Sucker Pygmy Octopus.kicad_pcb (KiCad board)
At the start: 2 copper layers, 73 x 55.9 mm, 51 parts, among them J1 DA15, J2 Molex, J3 PT 3-4, J4 PT 1-2, J5 Enable, J6 Pin Header, Q1 STN3NF06, Q2 STN3NF06, Q3 STN3NF06, Q4 STN3NF06, Q5 STN3NF06

Commit message: .
Parts:
- removed D1, D11, D12, D13, D2, D3, D4, D5: SBR130S3-7, Diode_SMD:D_SOD-323_HandSoldering
- removed D10, D6, D7, D8, D9: Red, LED_SMD:LED_0805_2012Metric_Pad1.15x1.40mm_HandSolder
- removed K1, K2, K3, K4, K5, K6, K7, K8: ~, Relay_THT:Relay_DPDT_Omron_G6K-2P
- Q1, Q2, Q3, Q4, Q5: value STN3NF06 -> Q_NMOS_DGS
- R10, R12, R18: value 10k -> 0.1
- R11, R17, R9: value 1k -> 500
- R16, R6: value 10k -> 1k
- R4: value 1k -> 0.1
Connections:
- Q1 pad 1: Net-(Q1-G) -> Net-(Q1-D)
- Q1 pad 2: /Relay_1 -> Net-(Q1-G)
- Q1 pad 3: GND -> Net-(Q1-S)
- Q2 pad 1: Net-(Q2-G) -> Net-(Q10-D)
- Q2 pad 2: /Relay_2 -> Net-(Q2-G)
- Q2 pad 3: GND -> Net-(Q10-S)
- Q3 pad 1: Net-(Q3-G) -> Net-(Q1-D)
- Q3 pad 2: /Relay_3 -> Net-(Q3-G)
- Q3 pad 3: GND -> Net-(Q1-S)
- Q4 pad 1: Net-(Q4-G) -> Net-(Q10-D)
- Q4 pad 2: /Relay_4 -> Net-(Q4-G)
- Q4 pad 3: GND -> Net-(Q10-S)
- Q5 pad 1: Net-(Q5-G) -> Net-(Q1-D)
- Q5 pad 2: /Relay_5 -> Net-(Q5-G)
- Q5 pad 3: GND -> Net-(Q1-S)
- R10 pad 1: /Relay_2_en -> Net-(Q1-S)
- R11 pad 1: /Relay_3_en -> Net-(U3C--)
- R11 pad 2: Net-(D8-A) -> Net-(Q10-S)
- R12 pad 1: /Relay_3_en -> Net-(Q10-S)
- R13 pad 1: /Relay_4_en -> Net-(C3-Pad1)
- R13 pad 2: Net-(Q4-G) -> Net-(Q5-G)
- R14 pad 1: /Relay_5_en -> Net-(C4-Pad1)
- R14 pad 2: Net-(Q5-G) -> Net-(Q6-G)
- R15 pad 1: /Relay_4_en -> Net-(C3-Pad1)
- R16 pad 1: /Relay_4_en -> Net-(C4-Pad1)
- R16 pad 2: GND -> Net-(Q8-G)
- R17 pad 1: /Relay_5_en -> Net-(U2D--)
- R17 pad 2: Net-(D10-A) -> Net-(Q1-S)
- R18 pad 1: /Relay_5_en -> Net-(Q1-S)
- R4 pad 1: /Relay_1_en -> Net-(Q10-S)
- R4 pad 2: Net-(Q1-G) -> GND
- R5 pad 1: /Relay_1_en -> Net-(C1-Pad1)
- R5 pad 2: Net-(D6-A) -> Net-(Q1-G)
- R6 pad 1: /Relay_1_en -> Net-(C2-Pad1)
- R6 pad 2: GND -> Net-(Q2-G)
- R7 pad 1: /Relay_2_en -> Net-(C1-Pad1)
- R7 pad 2: Net-(Q2-G) -> Net-(Q3-G)
- R8 pad 1: /Relay_3_en -> Net-(C2-Pad1)
- R8 pad 2: Net-(Q3-G) -> Net-(Q4-G)
- R9 pad 1: /Relay_2_en -> Net-(U2C--)
- R9 pad 2: Net-(D7-A) -> Net-(Q1-S)
Routing:
- net Net-(Q5-G): track 36.3 -> 71.6 mm, vias 1 -> 2
- net GND: track 0.00 -> 35.1 mm, vias 2 -> 3
- net Net-(Q3-G): track 8.09 -> 35.3 mm, vias 1 -> 2
- net Net-(Q1-G): track 35.1 -> 16.2 mm, vias 1 -> 0
- net /Relay_4: track 17.0 -> 0.00 mm
- net /Relay_1: track 16.4 -> 0.00 mm
- net /Relay_5: track 16.4 -> 0.00 mm
- net /Relay_2: track 16.4 -> 0.00 mm
- net (no net): track 0.00 -> 12.7 mm
- net /Relay_3: track 12.4 -> 0.00 mm, vias 1 -> 0
- net Net-(Q2-G): track 22.9 -> 13.2 mm, vias 1 -> 0
- net Net-(Q1-S): track 0.00 -> 6.11 mm
- net Net-(Q10-S): track 0.00 -> 3.05 mm
- net Net-(D8-A): track 3.05 -> 0.00 mm
- net Net-(D7-A): track 3.05 -> 0.00 mm
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