File: KiCAD/CIB - Star-Sucker Pygmy Octopus.kicad_sch (KiCad schematic)
At the start: 63 parts, among them J1 DA15, J2 Molex, J3 PT 3-4, J4 PT 1-2, J5 Enable, J6 Pin Header

Commit message: .
Parts:
- gave numbers to parts that had none: 45
Other:
- note removed: "https://chargepoint.atlassian.net/wiki/spaces/EN/pages/5094740380/Pygmy+Octopus"

Commit message: .
Parts:
- removed J1: DA15, Connector_Dsub:DSUB-9_Female_Horizontal_P2.77x2.84mm_EdgePinOffset7.70mm_Housed_MountingHolesOffset9.12mm, symbol Connector:DE9_Receptacle_MountingHoles
- removed J2: Molex, Connector_Molex:Molex_Micro-Fit_3.0_43045-1018_2x05-1MP_P3.00mm_Vertical, symbol Connector_Generic:Conn_02x05_Top_Bottom
- removed J3: PT 3-4, TerminalBlock_Phoenix:TerminalBlock_Phoenix_MPT-0,5-4-2.54_1x04_P2.54mm_Horizontal, symbol Connector:Screw_Terminal_01x04
- removed J4: PT 1-2, TerminalBlock_Phoenix:TerminalBlock_Phoenix_MPT-0,5-4-2.54_1x04_P2.54mm_Horizontal, symbol Connector:Screw_Terminal_01x04
- removed J5: Enable, Connector_Molex:Molex_Micro-Fit_3.0_43045-1218_2x06-1MP_P3.00mm_Vertical, symbol Connector_Generic:Conn_02x06_Top_Bottom
- removed J6: Pin Header, Connector_PinHeader_2.54mm:PinHeader_2x05_P2.54mm_Vertical, symbol Connector:Conn_01x10_Pin
Other:
- note removed: "Swap this out for a D25"
- moved on the sheet: U3E
